File: handle/fer_a_souder.kicad_pcb (KiCad board)
At the start: 2 copper layers, 42 parts, among them CON1 AVR-ISP-6, CON2 AVR-ISP-6, IC1 ATMEGA328P-A, IC2 ATTINY85-S, K1 CONN_3, P1 CONN_2, P2 CONN_5, P3 CONN_4, P4 CONN_4, U1 7805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

Commit message: Swapped folders
Parts:
- removed C10, C13, C14: 1n, SM1206
- removed C11: 200n, SM1206
- removed C12, C15, C17, C7: 1u, SM1206
- removed C16, C18, C8: 100u, SMD2917
- removed CON1, CON2: AVR-ISP-6, pin_array_3x2
- removed D1, D2: DIODESCH, SMD2917
- removed D5: DIODE, SM1206
- removed IC1: ATMEGA328P-A, TQFP32
- removed IC2: ATTINY85-S, SOIC-8
- removed K1: CONN_3, PIN_ARRAY_3X1
- removed L1, L2: 47u, INDCMS12.5
- removed TrouFixation2.1mm (x3): P***, trouFixation3.1mm
- removed svg2mod-rev: G***, svg2mod-rev
- added P10: CONN_1, pinCMD, F.Cu at (25.3, 18.4)
- added P11: CONN_1, pinCMD, B.Cu at (25.3, 18.4)
- added P12: CONN_1, pinCMD, F.Cu at (17.4, 23.6)
- added P13: CONN_1, pinCMD, F.Cu at (25.3, 23.4)
- added P5: CONN_1, pinCMD, B.Cu at (30.9, 18.4)
- added P6: CONN_1, pinCMD, B.Cu at (32.0, 19.1)
- added R4: 8k2, SM0603, F.Cu at (16.6, 19.3)
- added R5: 680k, SM0603, F.Cu at (18.2, 19.3)
- added R6: R, SM0603, F.Cu at (30.2, 22.1)
- added R7: R, SM0603, F.Cu at (31.7, 22.1)
- added R8: R, SM0603, F.Cu at (30.7, 19.6)
- added U4: MCP3221, SOT23-5, F.Cu at (20.8, 19.7)
- C1: value 1u -> 10u; footprint SM1206 -> SM0603
- C2: footprint SM1206 -> SM0603
- C3, C6: value 1u -> 0.1u; footprint SM1206 -> SM0603
- C4: value CAPAPOL -> 0.1u; footprint SMD2917 -> SM0603
- C5: value 100u -> 1u; footprint SMD2917 -> SM0603
- P1: value CONN_2 -> CONN_1; footprint PIN_ARRAY_2X1 -> pinCMD
- P2: value CONN_5 -> CONN_1; footprint PIN_ARRAY_5x1 -> pinCMD; moved to B.Cu
- P3, P4: value CONN_4 -> CONN_1; footprint PIN_ARRAY_4x1 -> pinCMD
- R1: value 10k -> 75k; footprint SM1206 -> SM0603; moved to B.Cu
- R2: value 2.2k -> 3.3M; footprint SM1206 -> SM0603
- R3: value 2.2k -> 10k; footprint SM1206 -> SM0603
- U1: value 7805 -> MCP1804-SOT235; footprint sot89 -> SOT23-5; moved to B.Cu
- U2: value LM5106 -> MMA8452Q; footprint msoic-10 -> QFN-16; moved to B.Cu
- U3: value ACS712 -> INA331; footprint so-8 -> MSOP_8; moved to B.Cu
- U5: value FDS6898A -> MPR121; footprint so-8 -> QFN20; moved to B.Cu
- moved U3 53.4 mm to (17.3, 21.1), turned to 0 degrees
- moved C6 50.9 mm to (21.6, 22.6), turned to 270 degrees
- moved C5 48.7 mm to (28.7, 22.4), turned to 90 degrees
- moved C1 44.9 mm to (20.1, 22.6), turned to 90 degrees
- moved U5 40.1 mm to (29.3, 20.9), turned to 0 degrees
- moved C4 38.7 mm to (24.1, 20.7), turned to 90 degrees
- moved U2 37.0 mm to (25.0, 20.8), turned to 0 degrees
- moved R3 35.4 mm to (16.6, 22.4), turned to 90 degrees
- moved P2 33.2 mm to (25.3, 23.4), turned to 90 degrees
- moved R2 32.6 mm to (18.2, 22.4), turned to 90 degrees
- moved U1 32.4 mm to (20.8, 22.2), turned to 90 degrees
- moved R1 30.3 mm to (28.9, 18.5)
- moved C3 28.9 mm to (29.2, 19.6)
- moved C2 24.1 mm to (25.7, 20.7)
- moved P4 23.9 mm to (30.7, 18.3), turned to 0 degrees
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Connections:
- C1 pad 1: +3.3V -> +12V
- C2 pad 1: +12V -> +3.3V
- C3 pad 1: +3.3V -> N-000003
- C4 pad 1: +12V -> N-0000024
- C5 pad 1: N-0000025 -> +3.3V
- P1 pad 1: GND -> /B
- P2 pad 1: /resistance -> +12V
- P3 pad 1: /SCK_2 -> /G
- P4 pad 1: /p -> /R
- R1 pad 1: N-000003 -> GND
- R1 pad 2: GND -> N-000002
- R2 pad 1: +3.3V -> /thermocouple
- R2 pad 2: /MOSI2 -> +3.3V
- R3 pad 1: +3.3V -> /thermocouple
- R3 pad 2: /SCK_2 -> N-0000034
- U2 pad 1: +12V -> +3.3V
- U2 pad 10: N-000007 -> GND
- U2 pad 2: N-000002 -> N-0000024
- U2 pad 3: N-000004 -> (no net)
- U2 pad 4: N-0000022 -> /SCL
- U2 pad 5: (no net) -> GND
- U2 pad 6: N-000003 -> /SDA
- U2 pad 7: /pont_en -> GND
- U2 pad 8: /MISO2 -> (no net)
- U2 pad 9: GND -> (no net)
- U3 pad 1: N-0000024 -> N-0000033
- U3 pad 2: N-0000024 -> GND
- U3 pad 3: /resistance -> N-0000034
- U3 pad 4: /resistance -> GND
- U3 pad 6: (no net) -> N-0000035
- U3 pad 7: /ISENS -> +3.3V
- U5 pad 1: GND -> (no net)
- U5 pad 2: N-000007 -> /SCL
- U5 pad 3: N-0000022 -> /SDA
- U5 pad 4: N-000004 -> /SDA
- U5 pad 5: +12V -> N-000003
- U5 pad 6: +12V -> GND
- U5 pad 7: N-0000022 -> N-000002
- U5 pad 8: N-0000022 -> (no net)
Routing:
- net GND: track 267.0 -> 46.6 mm, vias 14 -> 7
- net N-0000022: track 171.8 -> 0.00 mm
- net +12V: track 153.8 -> 16.2 mm, vias 4 -> 1
- net N-0000024: track 127.3 -> 1.35 mm, vias 6 -> 1
- net N-0000025: track 82.5 -> 0.00 mm, vias 2 -> 0
- net +3.3V: track 110.0 -> 33.4 mm
- net /SCK_2: track 62.9 -> 0.00 mm, vias 3 -> 0
- net /MOSI2: track 54.5 -> 0.00 mm, vias 3 -> 0
- net N-000004: track 32.3 -> 0.00 mm
- net N-000002: track 29.1 -> 1.45 mm
- net /resistance: track 22.3 -> 0.00 mm, vias 2 -> 0
- net /MISO: track 17.6 -> 0.00 mm, vias 1 -> 0
- net /SCK: track 16.6 -> 0.00 mm, vias 1 -> 0
- net N-000007: track 15.8 -> 0.00 mm
- net /SDA: track 0.00 -> 15.7 mm, vias 0 -> 3
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Other:
- net class Default: via_dia 0.6858 -> 0.6096
- rule via_min_drill: 0.3302 -> 0.254
- rule via_min_size: 0.6858 -> 0.4572
- board text added: "+12"
- board text added: "J. Besse WMRP 6.2"
- board text removed: "+"
- board text removed: "-ISP Attiny"
- board text removed: "12V"
- board text removed: "12V-"
- board text removed: "3.3V"
- board text removed: "Heat"
- board text removed: "ISP 328p-"
- board text removed: "MISO"
- board text removed: "MOSI"
- board text removed: "OLED-"
- board text removed: "Rx"
- board text removed: "SCK"
- board text removed: "Station WMRP rev 6.2 Julien BESSE"
- board text removed: "Tx"
- board text removed: "UART-"
- board text removed: "bp"
- board text removed: "encodeur"
- board text removed: "fer a souder"
- board text removed: "r+"
- board text removed: "r-"
- board text removed: "~RST"
