File: handle/fer_a_souder.sch (KiCad schematic (older format))
At the start: 39 parts, among them CON1 AVR-ISP-6, CON2 AVR-ISP-6, IC1 ATMEGA328P-A, IC2 ATTINY85-S, K1 CONN_3, P1 CONN_2, P2 CONN_5, P3 CONN_4, P4 CONN_4, U1 7805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

Commit message: Swapped folders
Parts:
- removed C1, C12, C15, C17, C7: 1u, ~, symbol C
- removed C10, C13, C14: 1n, ~, symbol C
- removed C11: 200n, ~, symbol C
- removed C16, C18, C5, C8: 100u, ~, symbol CAPAPOL
- removed C4: CAPAPOL, ~, symbol CAPAPOL
- removed CON1, CON2: AVR-ISP-6, AVR-ISP-6, symbol AVR-ISP-6
- removed D1, D2: DIODESCH, ~, symbol DIODESCH
- removed D5: DIODE, ~, symbol DIODE
- removed IC1: ATMEGA328P-A, TQFP32, symbol ATMEGA328P-A
- removed IC2: ATTINY85-S, SO8-200, symbol ATTINY85-S
- removed K1: CONN_3, symbol CONN_3
- removed L1, L2: 47u, ~, symbol INDUCTOR
- removed LOGO1: LOGO, symbol CONN_1
- removed P1: CONN_2, symbol CONN_2
- removed P2: CONN_5, symbol CONN_5
- removed P3, P4: CONN_4, ~, symbol CONN_4
- removed U1: 7805, ~, symbol 7805
- removed U2: LM5106, ~, symbol LM5106
- removed U3: ACS712, ~, symbol ACS712
- removed U5: FDS6898A, ~, symbol FDS6898A
- added C2, C5: 1u, ~, symbol C
- added C4: 0.1u, ~, symbol C
- added P1, P10, P11, P12, P13, P2, P3, P4, P5, P6: CONN_1, symbol CONN_1
- added R4: 8k2, ~, symbol R
- added R5: 680k, ~, symbol R
- added R6, R7, R8: R, ~, symbol R
- added U1: MCP1804-SOT235, SOT-23-5, symbol MCP1804-SOT235
- added U2: MMA8452Q, symbol MMA8452Q
- added U3: INA331, ~, symbol INA331
- added U4: MCP3221, ~, symbol MCP3221
- added U5: MPR121, ~, symbol MPR121
- C1: renamed from C2; value 1u -> 10u
- C3, C6: value 1u -> 0.1u
- R1: value 10k -> 75k
- R2: value 2.2k -> 3.3M
- R3: value 2.2k -> 10k
Connections:
- net labels added: B, G, R, T1, T2, thermocouple
- net labels removed: ISENS, MISO, MISO2, MOSI, MOSI2, RST, RST_2, RXD, SCK, SCK_2, TXD, p, pont_en, pont_in, r+, r-, resistance
- wire segments 152 -> 82
- no-connect marks 16 -> 11
Other:
- note added: "Adresse 0x5C -->"
- note added: "Thermocouple"
- note added: "Vers la\n base"
- note removed: "http://fr.rs-online.com/web/p/condensateurs-tantale/6844471/"
- note removed: "http://fr.rs-online.com/web/p/inductances-cms-bobinees/7701047/\n"
- moved on the sheet: C1
