File: station/fer_a_souder.kicad_pcb (KiCad board)
At the start: 2 copper layers, 29 parts, among them P1 CONN_1, P10 CONN_1, P11 CONN_1, P12 CONN_1, P13 CONN_1, P2 CONN_1, P3 CONN_1, P4 CONN_1, P5 CONN_1, P6 CONN_1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

Commit message: Swapped folders
Parts:
- removed P10, P11, P12, P13, P5, P6: CONN_1, pinCMD
- removed R4: 8k2, SM0603
- removed R5: 680k, SM0603
- removed R6, R7, R8: R, SM0603
- removed U4: MCP3221, SOT23-5
- added C10: 1n, SM1206, F.Cu at (37.4, 46.4)
- added C11: 200n, SM1206, F.Cu at (48.8, 34.4)
- added C12: 1u, SM1206, F.Cu at (55.7, 35.5)
- added C13: 1n, SM1206, F.Cu at (37.4, 43.8)
- added C14: 1n, SM1206, F.Cu at (37.4, 41.3)
- added C15: 1u, SM1206, F.Cu at (85.6, 28.1)
- added C16: 100u, SMD2917, F.Cu at (81.8, 30.6)
- added C17: 1u, SM1206, F.Cu at (85.6, 33.9)
- added C18: 100u, SMD2917, F.Cu at (94.5, 30.6)
- added C7: 1u, SM1206, F.Cu at (42.7, 41.3)
- added C8: 100u, SMD2917, F.Cu at (89.4, 30.6)
- added CON1: AVR-ISP-6, pin_array_3x2, F.Cu at (31.5, 33.2)
- added CON2: AVR-ISP-6, pin_array_3x2, F.Cu at (48.0, 43.3)
- added D1: DIODESCH, SMD2917, F.Cu at (66.6, 30.6)
- added D2: DIODESCH, SMD2917, F.Cu at (71.7, 30.6)
- added D5: DIODE, SM1206, F.Cu at (51.6, 34.4)
- added IC1: ATMEGA328P-A, TQFP32, F.Cu at (40.7, 33.4)
- added IC2: ATTINY85-S, SOIC-8, F.Cu at (55.7, 45.9)
- added K1: CONN_3, PIN_ARRAY_3X1, F.Cu at (32.8, 28.1)
- added L1: 47u, INDCMS12.5, F.Cu at (76.0, 44.0)
- added L2: 47u, INDCMS12.5, F.Cu at (90.0, 44.0)
- added TrouFixation2.1mm: P***, trouFixation3.1mm, F.Cu at (100.0, 28.4)
- added TrouFixation2.1mm: P***, trouFixation3.1mm, F.Cu at (100.0, 47.4)
- added TrouFixation2.1mm: P***, trouFixation3.1mm, F.Cu at (29.0, 47.4)
- added svg2mod-rev: G***, svg2mod-rev, F.Cu at (81.9, -25.5)
- C1: value 10u -> 1u; footprint SM0603 -> SM1206
- C2: footprint SM0603 -> SM1206
- C3, C6: value 0.1u -> 1u; footprint SM0603 -> SM1206
- C4: value 0.1u -> CAPAPOL; footprint SM0603 -> SMD2917
- C5: value 1u -> 100u; footprint SM0603 -> SMD2917
- P1: value CONN_1 -> CONN_2; footprint pinCMD -> PIN_ARRAY_2X1
- P2: value CONN_1 -> CONN_5; footprint pinCMD -> PIN_ARRAY_5x1; moved to F.Cu
- P3, P4: value CONN_1 -> CONN_4; footprint pinCMD -> PIN_ARRAY_4x1
- R1: value 75k -> 10k; footprint SM0603 -> SM1206; moved to F.Cu
- R2: value 3.3M -> 2.2k; footprint SM0603 -> SM1206
- R3: value 10k -> 2.2k; footprint SM0603 -> SM1206
- U1: value MCP1804-SOT235 -> 7805; footprint SOT23-5 -> sot89; moved to F.Cu
- U2: value MMA8452Q -> LM5106; footprint QFN-16 -> msoic-10; moved to F.Cu
- U3: value INA331 -> ACS712; footprint MSOP_8 -> so-8; moved to F.Cu
- U5: value MPR121 -> FDS6898A; footprint QFN20 -> so-8; moved to F.Cu
- moved U3 53.4 mm to (64.5, 45.9), turned to 90 degrees
- moved C6 50.9 mm to (64.6, 49.9), turned to 180 degrees
- moved C5 48.7 mm to (76.7, 30.6), turned to 270 degrees
- moved C1 44.9 mm to (55.7, 49.9), turned to 0 degrees
- moved U5 40.1 mm to (64.5, 40.0), turned to 270 degrees
- moved C4 38.7 mm to (61.5, 30.6), turned to 270 degrees
- moved U2 37.0 mm to (56.7, 40.0), turned to 270 degrees
- moved R3 35.4 mm to (42.7, 46.4), turned to 180 degrees
- moved P2 33.2 mm to (45.5, 49.7), turned to 180 degrees
- moved R2 32.6 mm to (42.7, 43.8), turned to 180 degrees
- moved U1 32.4 mm to (52.9, 27.3), turned to 0 degrees
- moved R1 30.3 mm to (55.6, 32.8)
- moved C3 28.9 mm to (56.9, 27.6)
- moved C2 24.1 mm to (48.8, 27.6)
- moved P4 23.9 mm to (32.8, 42.1), turned to 90 degrees
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Connections:
- C1 pad 1: +12V -> +3.3V
- C2 pad 1: +3.3V -> +12V
- C3 pad 1: N-000003 -> +3.3V
- C4 pad 1: N-0000024 -> +12V
- C5 pad 1: +3.3V -> N-0000025
- P1 pad 1: /B -> GND
- P2 pad 1: +12V -> /resistance
- P3 pad 1: /G -> /SCK_2
- P4 pad 1: /R -> /p
- R1 pad 1: GND -> N-000003
- R1 pad 2: N-000002 -> GND
- R2 pad 1: /thermocouple -> +3.3V
- R2 pad 2: +3.3V -> /MOSI2
- R3 pad 1: /thermocouple -> +3.3V
- R3 pad 2: N-0000034 -> /SCK_2
- U2 pad 1: +3.3V -> +12V
- U2 pad 10: GND -> N-000007
- U2 pad 2: N-0000024 -> N-000002
- U2 pad 3: (no net) -> N-000004
- U2 pad 4: /SCL -> N-0000022
- U2 pad 5: GND -> (no net)
- U2 pad 6: /SDA -> N-000003
- U2 pad 7: GND -> /pont_en
- U2 pad 8: (no net) -> /MISO2
- U2 pad 9: (no net) -> GND
- U3 pad 1: N-0000033 -> N-0000024
- U3 pad 2: GND -> N-0000024
- U3 pad 3: N-0000034 -> /resistance
- U3 pad 4: GND -> /resistance
- U3 pad 6: N-0000035 -> (no net)
- U3 pad 7: +3.3V -> /ISENS
- U5 pad 1: (no net) -> GND
- U5 pad 2: /SCL -> N-000007
- U5 pad 3: /SDA -> N-0000022
- U5 pad 4: /SDA -> N-000004
- U5 pad 5: N-000003 -> +12V
- U5 pad 6: GND -> +12V
- U5 pad 7: N-000002 -> N-0000022
- U5 pad 8: (no net) -> N-0000022
Routing:
- net GND: track 46.6 -> 267.0 mm, vias 7 -> 14
- net N-0000022: track 0.00 -> 171.8 mm
- net +12V: track 16.2 -> 153.8 mm, vias 1 -> 4
- net N-0000024: track 1.35 -> 127.3 mm, vias 1 -> 6
- net N-0000025: track 0.00 -> 82.5 mm, vias 0 -> 2
- net +3.3V: track 33.4 -> 110.0 mm
- net /SCK_2: track 0.00 -> 62.9 mm, vias 0 -> 3
- net /MOSI2: track 0.00 -> 54.5 mm, vias 0 -> 3
- net N-000004: track 0.00 -> 32.3 mm
- net N-000002: track 1.45 -> 29.1 mm
- net /resistance: track 0.00 -> 22.3 mm, vias 0 -> 2
- net /MISO: track 0.00 -> 17.6 mm, vias 0 -> 1
- net /SCK: track 0.00 -> 16.6 mm, vias 0 -> 1
- net N-000007: track 0.00 -> 15.8 mm
- net /SDA: track 15.7 -> 0.00 mm, vias 3 -> 0
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Other:
- net class Default: via_dia 0.6096 -> 0.6858
- rule via_min_drill: 0.254 -> 0.3302
- rule via_min_size: 0.4572 -> 0.6858
- board text added: "+"
- board text added: "-ISP Attiny"
- board text added: "12V"
- board text added: "12V-"
- board text added: "3.3V"
- board text added: "Heat"
- board text added: "ISP 328p-"
- board text added: "MISO"
- board text added: "MOSI"
- board text added: "OLED-"
- board text added: "Rx"
- board text added: "SCK"
- board text added: "Station WMRP rev 6.2 Julien BESSE"
- board text added: "Tx"
- board text added: "UART-"
- board text added: "bp"
- board text added: "encodeur"
- board text added: "fer a souder"
- board text added: "r+"
- board text added: "r-"
- board text added: "~RST"
- board text removed: "+12"
- board text removed: "J. Besse WMRP 6.2"
