File: station/fer_a_souder.sch (KiCad schematic (older format))
At the start: 29 parts, among them P1 CONN_1, P10 CONN_1, P11 CONN_1, P12 CONN_1, P13 CONN_1, P2 CONN_1, P3 CONN_1, P4 CONN_1, P5 CONN_1, P6 CONN_1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

Commit message: Swapped folders
Parts:
- removed C2, C5: 1u, ~, symbol C
- removed C4: 0.1u, ~, symbol C
- removed P1, P10, P11, P12, P13, P2, P3, P4, P5, P6: CONN_1, symbol CONN_1
- removed R4: 8k2, ~, symbol R
- removed R5: 680k, ~, symbol R
- removed R6, R7, R8: R, ~, symbol R
- removed U1: MCP1804-SOT235, SOT-23-5, symbol MCP1804-SOT235
- removed U2: MMA8452Q, symbol MMA8452Q
- removed U3: INA331, ~, symbol INA331
- removed U4: MCP3221, ~, symbol MCP3221
- removed U5: MPR121, ~, symbol MPR121
- added C1, C12, C15, C17, C7: 1u, ~, symbol C
- added C10, C13, C14: 1n, ~, symbol C
- added C11: 200n, ~, symbol C
- added C16, C18, C5, C8: 100u, ~, symbol CAPAPOL
- added C4: CAPAPOL, ~, symbol CAPAPOL
- added CON1, CON2: AVR-ISP-6, AVR-ISP-6, symbol AVR-ISP-6
- added D1, D2: DIODESCH, ~, symbol DIODESCH
- added D5: DIODE, ~, symbol DIODE
- added IC1: ATMEGA328P-A, TQFP32, symbol ATMEGA328P-A
- added IC2: ATTINY85-S, SO8-200, symbol ATTINY85-S
- added K1: CONN_3, symbol CONN_3
- added L1, L2: 47u, ~, symbol INDUCTOR
- added LOGO1: LOGO, symbol CONN_1
- added P1: CONN_2, symbol CONN_2
- added P2: CONN_5, symbol CONN_5
- added P3, P4: CONN_4, ~, symbol CONN_4
- added U1: 7805, ~, symbol 7805
- added U2: LM5106, ~, symbol LM5106
- added U3: ACS712, ~, symbol ACS712
- added U5: FDS6898A, ~, symbol FDS6898A
- C2: renamed from C1; value 10u -> 1u
- C3, C6: value 0.1u -> 1u
- R1: value 75k -> 10k
- R2: value 3.3M -> 2.2k
- R3: value 10k -> 2.2k
Connections:
- net labels added: ISENS, MISO, MISO2, MOSI, MOSI2, RST, RST_2, RXD, SCK, SCK_2, TXD, p, pont_en, pont_in, r+, r-, resistance
- net labels removed: B, G, R, T1, T2, thermocouple
- wire segments 82 -> 152
- no-connect marks 11 -> 16
Other:
- note added: "http://fr.rs-online.com/web/p/condensateurs-tantale/6844471/"
- note added: "http://fr.rs-online.com/web/p/inductances-cms-bobinees/7701047/\n"
- note removed: "Adresse 0x5C -->"
- note removed: "Thermocouple"
- note removed: "Vers la\n base"
- moved on the sheet: C2
